File: Starter_x51_USB.sch (KiCad schematic (older format))
At the start: 50 parts, among them CON1 BARREL_JACK, CON2 USB-MINI-B, IC1 LM1117, P1 CONN_01X03, P10 CONN_01X01, P11 CONN_01X01, P12 CONN_01X01, P13 CONN_01X04, P2 CONN_01X03, P3 CONN_01X03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

Commit message: routing
Parts:
- removed Q1: BC557, TO92, symbol BC557
- added Q?: PNP, symbol PNP
Connections:
- net D4: now also P7.5 (P5), RR1.6, U2.35 (P0.4(AD4)); no longer P6.4 (P4), U2.25 (P2.4(A12))
- net D5: now also P7.6 (P6), RR1.7, U2.34 (P0.5(AD5)); no longer P6.3 (P3), U2.26 (P2.5(A13))
- net D6: now also P7.7 (P7), RR1.8, U2.33 (P0.6(AD6)); no longer P6.2 (P2), U2.27 (P2.6(A14))
- net D7: now also P7.8 (P8), RR1.9, U2.32 (P0.7(AD7)); no longer P6.1 (P1), U2.28 (P2.7(A15))
- net E: now also P7.3 (P3), RR1.4, U2.37 (P0.2(AD2)); no longer P6.6 (P6), U2.23 (P2.2(A10))
- net GND: now also C4.2, C5.2
- net R/W: now also P7.2 (P2), RR1.3, U2.38 (P0.1(AD1)); no longer P6.7 (P7), U2.22 (P2.1(A9))
- net RS: now also P7.1 (P1), RR1.2, U2.39 (P0.0(AD0)); no longer P6.8 (P8), U2.21 (P2.0(A8))
- net VCC: now also C2.1, IC1.2 (OUT), IC1.4 (OUT), R5.2, Q?.1 (E)
- net at R2.1, R3.2: now also Q?.2 (B)
- net at R4.2: now also Q?.3 (C)
- new net: P6.8 (P8), U2.21 (P2.0(A8))
- new net: P6.7 (P7), U2.22 (P2.1(A9))
- new net: P6.6 (P6), U2.23 (P2.2(A10))
- new net: P6.4 (P4), U2.25 (P2.4(A12))
- new net: P6.3 (P3), U2.26 (P2.5(A13))
- new net: P6.2 (P2), U2.27 (P2.6(A14))
- new net: P6.1 (P1), U2.28 (P2.7(A15))
Changed lines of the file:
@@
 L GND #PWR04
 U 1 1 56373DB8
-P 7900 3500
-F 0 "#PWR04" H 7900 3250 60  0001 C CNN
-F 1 "GND" H 7900 3350 60  0000 C CNN
-F 2 "" H 7900 3500 60  0000 C CNN
-F 3 "" H 7900 3500 60  0000 C CNN
-	1    7900 3500
+P 7900 3550
+F 0 "#PWR04" H 7900 3300 60  0001 C CNN
+F 1 "GND" H 7900 3400 60  0000 C CNN
+F 2 "" H 7900 3550 60  0000 C CNN
+F 3 "" H 7900 3550 60  0000 C CNN
+	1    7900 3550
 	1    0    0    -1
 $EndComp
@@
 	1    1750 3250
 	-1   0    0    1
-$EndComp
-$Comp
-L BC557 Q1
-U 1 1 56374ED6
-P 2050 2950
-F 0 "Q1" H 2050 2801 40  0000 R CNN
-F 1 "BC557" H 2050 3100 40  0000 R CNN
-F 2 "TO92" H 1950 3052 29  0000 C CNN
-F 3 "" H 2050 2950 60  0000 C CNN
-	1    2050 2950
-	1    0    0    -1
 $EndComp
 Wire Wire Line
@@
 Wire Wire Line
 	10600 5550 10600 5600
-Text Label 7000 2150 0    50   ~ 0
+Text Label 7000 1400 0    50   ~ 0
 D4
-Text Label 7000 2050 0    50   ~ 0
+Text Label 7000 1500 0    50   ~ 0
 D5
-Text Label 7000 1950 0    50   ~ 0
+Text Label 7000 1600 0    50   ~ 0
 D6
-Text Label 7000 1850 0    50   ~ 0
+Text Label 7000 1700 0    50   ~ 0
 D7
-Text Label 7000 2550 0    50   ~ 0
+Text Label 7000 1000 0    50   ~ 0
 RS
-Text Label 7000 2450 0    50   ~ 0
+Text Label 7000 1100 0    50   ~ 0
 R/W
-Text Label 7000 2350 0    50   ~ 0
+Text Label 7000 1200 0    50   ~ 0
 E
 $Comp
@@
 Wire Wire Line
 	11100 1400 11100 1250
+Wire Wire Line
+	7900 3500 7900 3550
+Connection ~ 7900 3500
+$Comp
+L VCC #PWR026
+U 1 1 56405D2D
+P 3400 4500
+F 0 "#PWR026" H 3400 4350 60  0001 C CNN
+F 1 "VCC" H 3400 4650 60  0000 C CNN
+F 2 "" H 3400 4500 60  0000 C CNN
+F 3 "" H 3400 4500 60  0000 C CNN
+	1    3400 4500
+	1    0    0    -1
+$EndComp
+Wire Wire Line
+	3400 4600 3400 4500
+$Comp
+L PNP Q?
+U 1 1 5640B6F4
+P 2050 2950
+F 0 "Q?" H 2050 2800 50  0000 R CNN
+F 1 "PNP" H 2050 3100 50  0000 R CNN
+F 2 "" H 2050 2950 60  0000 C CNN
+F 3 "" H 2050 2950 60  0000 C CNN
+	1    2050 2950
+	1    0    0    -1
+$EndComp
 $EndSCHEMATC

Commit message: corrected files
Parts:
- gave numbers to parts that had none: 1
Changed lines of the file:
@@
 	3400 4600 3400 4500
 $Comp
-L PNP Q?
+L PNP Q1
 U 1 1 5640B6F4
 P 2050 2950
-F 0 "Q?" H 2050 2800 50  0000 R CNN
+F 0 "Q1" H 2050 2800 50  0000 R CNN
 F 1 "PNP" H 2050 3100 50  0000 R CNN
 F 2 "" H 2050 2950 60  0000 C CNN
