File: Starter_x51_USB.kicad_pcb (KiCad board)
At the start: 2 copper layers, 90 x 70 mm, 50 parts, among them CON1 BARREL_JACK, CON2 USB-MINI-B, IC1 LM1117, P1 CONN_01X03, P10 CONN_01X01, P11 CONN_01X01, P12 CONN_01X01, P13 CONN_01X04, P2 CONN_01X03, P3 CONN_01X03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

Commit message: routing
Parts:
- added LOGO: , logo:LOGO (1), B.Cu at (115.6, 72.8)
- moved P8 74.7 mm to (56.4, 75.2), turned to 90 degrees
- moved P13 41.2 mm to (127.9, 47.0), turned to 270 degrees
- moved R3 21.6 mm to (66.5, 79.2), turned to 0 degrees
- moved R1 21.3 mm to (66.5, 76.7), turned to 180 degrees
- moved R2 17.6 mm to (70.1, 78.0)
- moved C3 15.0 mm to (76.5, 65.0)
- moved R8 14.2 mm to (103.6, 66.0), turned to 270 degrees
- moved CON2 10.9 mm to (50.8, 56.4)
- moved R13 10.8 mm to (116.8, 94.5), turned to 270 degrees
- moved R12 10.7 mm to (114.3, 94.5), turned to 270 degrees
- moved R11 10.7 mm to (111.8, 94.5), turned to 270 degrees
- moved R10 10.7 mm to (109.2, 94.5), turned to 270 degrees
- moved C1 10.3 mm to (64.3, 71.6), turned to 180 degrees
- moved Q1 9.45 mm to (66.3, 84.8), turned to 315 degrees
- moved DS1 9.16 mm to (62.5, 57.9)
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Connections:
- C2 pad 1: Net-(C2-Pad1) -> VCC
- C4 pad 2: Net-(C4-Pad2) -> GND
- C5 pad 2: Net-(C4-Pad2) -> GND
- IC1 pad 2: Net-(C2-Pad1) -> VCC
- IC1 pad 4: Net-(C2-Pad1) -> VCC
- P6 pad 1: /D7 -> Net-(P6-Pad1)
- P6 pad 2: /D6 -> Net-(P6-Pad2)
- P6 pad 3: /D5 -> Net-(P6-Pad3)
- P6 pad 4: /D4 -> Net-(P6-Pad4)
- P6 pad 6: /E -> Net-(P6-Pad6)
- P6 pad 7: /R/W -> Net-(P6-Pad7)
- P6 pad 8: /RS -> Net-(P6-Pad8)
- P7 pad 1: Net-(P7-Pad1) -> /RS
- P7 pad 2: Net-(P7-Pad2) -> /R/W
- P7 pad 3: Net-(P7-Pad3) -> /E
- P7 pad 5: Net-(P7-Pad5) -> /D4
- P7 pad 6: Net-(P7-Pad6) -> /D5
- P7 pad 7: Net-(P7-Pad7) -> /D6
- P7 pad 8: Net-(P7-Pad8) -> /D7
- R5 pad 2: Net-(C2-Pad1) -> VCC
- RR1 pad 2: Net-(P7-Pad1) -> /RS
- RR1 pad 3: Net-(P7-Pad2) -> /R/W
- RR1 pad 4: Net-(P7-Pad3) -> /E
- RR1 pad 6: Net-(P7-Pad5) -> /D4
- RR1 pad 7: Net-(P7-Pad6) -> /D5
- RR1 pad 8: Net-(P7-Pad7) -> /D6
- RR1 pad 9: Net-(P7-Pad8) -> /D7
- U2 pad 21: /RS -> Net-(P6-Pad8)
- U2 pad 22: /R/W -> Net-(P6-Pad7)
- U2 pad 23: /E -> Net-(P6-Pad6)
- U2 pad 25: /D4 -> Net-(P6-Pad4)
- U2 pad 26: /D5 -> Net-(P6-Pad3)
- U2 pad 27: /D6 -> Net-(P6-Pad2)
- U2 pad 28: /D7 -> Net-(P6-Pad1)
- U2 pad 32: Net-(P7-Pad8) -> /D7
- U2 pad 33: Net-(P7-Pad7) -> /D6
- U2 pad 34: Net-(P7-Pad6) -> /D5
- U2 pad 35: Net-(P7-Pad5) -> /D4
- U2 pad 37: Net-(P7-Pad3) -> /E
- U2 pad 38: Net-(P7-Pad2) -> /R/W
- U2 pad 39: Net-(P7-Pad1) -> /RS
Routing:
- net GND: track 0.00 -> 390.1 mm, vias 0 -> 3
- net VCC: track 0.00 -> 386.0 mm, vias 0 -> 9
- net /RST: track 0.00 -> 167.0 mm, vias 0 -> 5
- net /TX: track 0.00 -> 158.1 mm
- net /RX: track 0.00 -> 155.5 mm, vias 0 -> 2
- net /Vin: track 0.00 -> 82.6 mm, vias 0 -> 1
- net /SCK: track 0.00 -> 74.5 mm, vias 0 -> 1
- net /MISO: track 0.00 -> 71.1 mm
- net /MOSI: track 0.00 -> 62.2 mm
- net Net-(P7-Pad4): track 0.00 -> 56.8 mm
- net /SW2: track 0.00 -> 54.3 mm
- net /SW1: track 0.00 -> 53.1 mm
- net Net-(DS1-Pad3): track 0.00 -> 43.3 mm, vias 0 -> 1
- net /R/W: track 0.00 -> 33.1 mm
- net /RS: track 0.00 -> 32.7 mm
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- added copper zone on B.Cu, net GND
- added copper zone on F.Cu, net VCC
Other:
- board text added: "ExploreEmbedded.com"
- board text added: "SW1(P3.2)"
- board text added: "SW2(P3.3)"
- board text removed: "SW1"
- board text removed: "SW2"

Commit message: corrected files
Parts:
- Q1: value BC557 -> PNP
- moved R4 1.17 mm to (66.0, 88.8)
Connections:
- Q1 pad 1: Net-(Q1-Pad1) -> VCC
- Q1 pad 3: VCC -> Net-(Q1-Pad3)
- R4 pad 2: Net-(Q1-Pad1) -> Net-(Q1-Pad3)
Routing:
- net VCC: track 386.0 -> 393.9 mm, vias 9 -> 8
- net Net-(Q1-Pad3): track 0.00 -> 5.03 mm
- net Net-(Q1-Pad1): track 5.00 -> 0.00 mm

Commit message: Final Design
Parts:
- added LOGO: , logo:LOGO (2), F.Cu at (56.4, 48.8)
Routing:
- net VCC: track 393.9 -> 420.1 mm
- net GND: track 390.1 -> 382.1 mm
Other:
- board text added: "->"
- board text added: "D4-P0.4 D5-P0.5 D6-P0.6 D7-P0.7"
- board text added: "Explore Stater 8051"
- board text added: "RS-P0.0 R/W-P0.1 E-P0.2"
- board text removed: "Stater 8051"
